File: PCB/Digital_Board/Digital_Board.kicad_pcb (KiCad board)
At the start: 2 copper layers, 101.6 x 53.3 mm, 19 parts, among them J1 Conn_01x08_Male, J2 Conn_01x08_Male, J3 Conn_01x08_Male, J4 Conn_02x18_Odd_Even, J5 Conn_02x03_Odd_Even, J6 Conn_01x10_Male, J7 Conn_01x08_Male, J8 Conn_01x08_Male, U1 LSM9DS1, U15 TMP36xS, U17 MMA1210, U18 SDCard

Commit message: Digital PCB update
Routing:
- net +3V3: track 74.1 -> 75.6 mm
Changed lines of the file:
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@@
     (thickness 1.6)
     (drawings 22)
-    (tracks 104)
+    (tracks 105)
     (zones 0)
     (modules 19)
@@
   )
   (setup
-    (last_trace_width 0.25)
+    (last_trace_width 0.508)
     (user_trace_width 0.127)
     (user_trace_width 0.254)
@@
   (segment (start 62.23 87.392) (end 62.23 74.93) (width 0.508) (layer B.Cu) (net 3))
   (segment (start 62.23 87.392) (end 63.208001 86.413999) (width 0.508) (layer B.Cu) (net 3))
-  (via (at 69.85 86.36) (size 0.8) (drill 0.4) (layers F.Cu B.Cu) (net 3))
-  (segment (start 82.55 86.36) (end 69.85 86.36) (width 0.508) (layer F.Cu) (net 3))
   (segment (start 63.262 86.36) (end 63.208001 86.413999) (width 0.508) (layer B.Cu) (net 3))
-  (segment (start 69.85 86.36) (end 63.262 86.36) (width 0.508) (layer B.Cu) (net 3))
   (segment (start 85.09 87.63) (end 93.98 87.63) (width 0.508) (layer F.Cu) (net 3))
   (segment (start 83.82 86.36) (end 85.09 87.63) (width 0.508) (layer F.Cu) (net 3))
   (segment (start 83.82 86.36) (end 86.605 86.36) (width 0.508) (layer F.Cu) (net 3))
+  (segment (start 62.23 87.392) (end 63.262 86.36) (width 0.508) (layer B.Cu) (net 3))
+  (via (at 64.77 86.36) (size 0.8) (drill 0.4) (layers F.Cu B.Cu) (net 3))
+  (segment (start 63.262 86.36) (end 64.77 86.36) (width 0.508) (layer B.Cu) (net 3))
   (segment (start 82.55 86.36) (end 83.82 86.36) (width 0.508) (layer F.Cu) (net 3))
+  (segment (start 64.77 86.36) (end 82.55 86.36) (width 0.508) (layer F.Cu) (net 3))
   (segment (start 109.855 80.9775) (end 110.49 81.6125) (width 0.254) (layer F.Cu) (net 5))
   (segment (start 109.855 74.675) (end 109.855 80.9775) (width 0.254) (layer F.Cu) (net 5))
